Commit message: Rebase from 'debian/noetic/leo_description'

File: urdf/macros.xacro (robot description, xacro)
@@ -64,5 +64,7 @@
     </xacro:macro>
     <!-- LINKS -->
-    <link name="${link_prefix}base_footprint"/>
+    <xacro:if value="${footprint_link}">
+      <link name="${link_prefix}base_footprint"/>
+    </xacro:if>
     <link name="${link_prefix}base_link">
       <inertial>
@@ -117,9 +119,11 @@
     <link name="${link_prefix}camera_optical_frame"/>
     <!-- JOINTS -->
-    <joint name="${joint_prefix}base_joint" type="fixed">
-      <origin xyz="0 0 0.19783" rpy="0 0 0"/>
-      <parent link="${link_prefix}base_footprint"/>
-      <child link="${link_prefix}base_link"/>
-    </joint>
+    <xacro:if value="${footprint_link}">
+      <joint name="${joint_prefix}base_joint" type="fixed">
+        <origin xyz="0 0 0.19783" rpy="0 0 0"/>
+        <parent link="${link_prefix}base_footprint"/>
+        <child link="${link_prefix}base_link"/>
+      </joint>
+    </xacro:if>
     <xacro:if value="${rockers_fixed}">
       <xacro:property name="rockers_joint_type" value="fixed"/>
