Commit message: Imported upstream version '1.2.2' of 'upstream'

File: leo_description/urdf/macros.xacro (robot description, xacro)
@@ -166,5 +166,5 @@
     </joint>
     <joint name="${joint_prefix}wheel_FR_joint" type="continuous">
-      <origin xyz="-0.15256 -0.08214 -0.08802" rpy="0 0 0"/>
+      <origin xyz="0.15256 -0.08214 -0.08802" rpy="0 0 0"/>
       <parent link="${link_prefix}rocker_R_link"/>
       <child link="${link_prefix}wheel_FR_link"/>
@@ -174,5 +174,5 @@
     </joint>
     <joint name="${joint_prefix}wheel_RR_joint" type="continuous">
-      <origin xyz="0.15256 -0.08214 -0.08802" rpy="0 0 0"/>
+      <origin xyz="-0.15256 -0.08214 -0.08802" rpy="0 0 0"/>
       <parent link="${link_prefix}rocker_R_link"/>
       <child link="${link_prefix}wheel_RR_link"/>

Commit message: Imported upstream version '2.0.1' of 'upstream'

File: leo_description/urdf/macros.xacro (robot description, xacro)
@@ -6,5 +6,6 @@
                        footprint_link:=true
                        link_prefix:=''
-                       joint_prefix:=''">
+                       joint_prefix:=''
+                       imu_translation:='0.0628 -0.0314 -0.0393'">
     <xacro:macro name="rocker_link" params="name">
       <link name="${link_prefix}rocker_${name}_link">
@@ -118,4 +119,5 @@
     <link name="${link_prefix}camera_frame"/>
     <link name="${link_prefix}camera_optical_frame"/>
+    <link name="${link_prefix}imu_frame"/>
     <!-- JOINTS -->
     <xacro:if value="${footprint_link}">
@@ -197,4 +199,9 @@
       <parent link="${link_prefix}camera_frame"/>
       <child link="${link_prefix}camera_optical_frame"/>
+    </joint>
+    <joint name="${joint_prefix}imu_joint" type="fixed">
+      <origin xyz="${imu_translation}" rpy="0 0 0"/>
+      <parent link="${link_prefix}base_link"/>
+      <child link="${link_prefix}imu_frame"/>
     </joint>
   </xacro:macro>
